File: payload_main_pcb/avionics-payload.sch (KiCad schematic (older format))
At the start: 29 parts, among them J1 Conn_Coaxial_x2, J2 Screw_Terminal_01x02, SW1 SW_Push, SW2 SW_Push, U1 ADXL357BEZ, U2 Teensy4.0, U3 RFM96W-433S2, U4 ublox_SAM-M8Q, U5 MS5607-02BA

Commit message: Added SD card
Parts:
- added J?: Micro_SD_Card, symbol Connector:Micro_SD_Card
Connections:
- net labels added: SD_3.3, SD_CLK, SD_CMD, SD_DAT0, SD_DAT1, SD_DAT2, SD_DAT3, SD_GND
- wire segments 118 -> 135
- no-connect marks 44 -> 30

Commit message: Work on ground station and new IMU added to payload
Parts:
- added R5, R6, R7: 10k, symbol Device:R
- added U7: ADIS16470AMLZ, footprints:ADIS16470AMLZ, symbol ADIS16470AMLZ:ADIS16470AMLZ
- C10: renamed from C?; value CP1 -> 3.3uF; footprint (none) -> Capacitor_Tantalum_SMD:CP_EIA-6032-15_Kemet-U_Pad2.25x2.35mm_HandSolder
- J1: renamed from J?; footprint (none) -> Connector_Card:microSD_HC_Wuerth_693072010801
- gave numbers to parts that had none: 9
- renumbered J1 to J2, J2 to J3, U4 to U5, U5 to U6
Connections:
- wire segments 135 -> 188
Other:
- moved on the sheet: C9, SW1, U6

Commit message: Added data module
Other:
- note added: "Data\n"

Commit message: Integrated ADIS16470 in schematic and removed ADXL357
Parts:
- removed C2, C5, C7: 1uF, Capacitor_SMD:C_0805_2012Metric_Pad1.15x1.40mm_HandSolder, symbol Device:C
- removed C3, C4, C6, C8: .1uF, Capacitor_SMD:C_0805_2012Metric_Pad1.15x1.40mm_HandSolder, symbol Device:C
- removed U1: ADXL357BEZ, footprints:ADXL357BEZ, symbol _ADXL357BEZ:ADXL357BEZ
- added SW1: SW_Push, Button_Switch_THT:SW_PUSH_6mm, symbol Switch:SW_Push
- C1: value 1uF -> 100nF; footprint Capacitor_SMD:C_0805_2012Metric_Pad1.15x1.40mm_HandSolder -> Capacitor_SMD:C_1206_3216Metric_Pad1.42x1.75mm_HandSolder
- C2: renamed from C9; footprint Capacitor_SMD:C_0805_2012Metric_Pad1.15x1.40mm_HandSolder -> Capacitor_SMD:C_1206_3216Metric_Pad1.42x1.75mm_HandSolder
- J3: footprint (none) -> Connector_PinSocket_2.54mm:PinSocket_2x01_P2.54mm_Vertical
- R1: renamed from R5; footprint (none) -> Resistor_SMD:R_1206_3216Metric_Pad1.42x1.75mm_HandSolder
- R2: renamed from R1; footprint Resistor_SMD:R_0805_2012Metric_Pad1.15x1.40mm_HandSolder -> Resistor_SMD:R_1206_3216Metric_Pad1.42x1.75mm_HandSolder
- R3: renamed from R2; footprint Resistor_SMD:R_0805_2012Metric_Pad1.15x1.40mm_HandSolder -> Resistor_SMD:R_1206_3216Metric_Pad1.42x1.75mm_HandSolder
- R4: renamed from R6; footprint (none) -> Resistor_SMD:R_1206_3216Metric_Pad1.42x1.75mm_HandSolder
- R5: renamed from R3; footprint Resistor_SMD:R_0805_2012Metric_Pad1.15x1.40mm_HandSolder -> Resistor_SMD:R_1206_3216Metric_Pad1.42x1.75mm_HandSolder
- R6: renamed from R4; footprint Resistor_SMD:R_0805_2012Metric_Pad1.15x1.40mm_HandSolder -> Resistor_SMD:R_1206_3216Metric_Pad1.42x1.75mm_HandSolder
- R7: footprint (none) -> Resistor_SMD:R_1206_3216Metric_Pad1.42x1.75mm_HandSolder
- renumbered C10 to C3, SW1 to SW2, SW2 to SW3, U7 to U1
Connections:
- net labels added: IMU_DR
- wire segments 188 -> 161
- no-connect marks 30 -> 26
Other:
- note removed: "Accelerometer"
- moved on the sheet: R1, U1, U2

Commit message: Lots of stuff
Parts:
- removed AE1: Antenna, symbol Device:Antenna
- removed D1, D2, D3, D4: LED, LED_SMD:LED_1206_3216Metric_Pad1.42x1.75mm_HandSolder, symbol Device:LED
- removed J2: Conn_Coaxial_x2, Connector_Coaxial:SMA_Amphenol_132134-14_Vertical, symbol Connector:Conn_Coaxial_x2
- added C2, C5, C6: 100nF, Capacitor_SMD:C_1206_3216Metric_Pad1.42x1.75mm_HandSolder, symbol Device:C
- added D1, D2, D3, D4: LED_RGBA, LED_SMD:LED_Avago_PLCC4_3.2x2.8mm_CW, symbol Device:LED_RGBA
- added J1: USB_C_Receptacle_USB2.0, Connector_USB:USB_C_Receptacle_GCT_USB4085, symbol Connector:USB_C_Receptacle_USB2.0
- added J3: Conn_Coaxial, Connector_Coaxial:SMA_Amphenol_132291_Vertical, symbol Connector:Conn_Coaxial
- added R10, R8: 51, Resistor_SMD:R_1206_3216Metric_Pad1.42x1.75mm_HandSolder, symbol Device:R
- added R11, R4, R9: 10, Resistor_SMD:R_1206_3216Metric_Pad1.42x1.75mm_HandSolder, symbol Device:R
- added U3: 74LS14, Package_DIP:DIP-14_W7.62mm_SMDSocket_SmallPads, symbol 74xx:74LS14
- C3: footprint Capacitor_Tantalum_SMD:CP_EIA-6032-15_Kemet-U_Pad2.25x2.35mm_HandSolder -> Capacitor_SMD:CP_Elec_10x10
- R2: value 220 -> R
- R3, R5: value 220 -> 51
- R6: value 220 -> 10
- SW1, SW2, SW3: footprint Button_Switch_THT:SW_PUSH_6mm -> Button_Switch_SMD:SW_SPST_FSMSM
- renumbered C2 to C4, J1 to J2, J3 to J4, R7 to R12, R4 to R7, U3 to U4, U4 to U5, U5 to U7
Connections:
- net +3V3: now also R2.1, C2.1, C5.1, C6.1, U3.14 (VCC)
- net GND: now also C2.2, C5.2, C6.2, D1.4 (A), D2.4 (A), D3.4 (A), D4.4 (A), J1.A1 (GND), J1.A12 (GND), J1.B1 (GND), J1.B12 (GND), J1.S1 (SHIELD), J3.2 (Ext), U3.7 (GND); no longer R2.1, R3.1, R5.1, R6.1
- net GPSStatus: now also U2.27 (20_A6_TX5_LRCLK1), R10.2, U3.1; no longer U2.4 (2_OUT2)
- net IMU_DR: now also U2.10 (8_TX2_IN1); no longer U2.28 (21_A7_RX5_BCLK1)
- net RX1: now also U2.23 (16_A2_RX4_SCL1); no longer U2.9 (7_RX2_OUT1A)
- net SensorStatus: now also R5.2, U2.29 (22_A8_CTX1), U3.9; no longer U2.5 (3_LRCLK2)
- net SystemStatus: now also R3.2, U2.30 (23_A9_CRX1_MCLK1), U3.5; no longer U2.7 (5_IN2)
- net TX1: now also U2.24 (17_A3_TX4_SDA1); no longer U2.10 (8_TX2_IN1)
- net TransmitterStatus: now also U2.28 (21_A7_RX5_BCLK1), R8.2, U3.3; no longer U2.6 (4_BCLK2)
- net at U4.9 (ANT): now also J3.1 (In)
- net V_USB: now reaches U2.34 (VUSB)
- net V_USB: now also J1.A4 (VBUS), J1.A9 (VBUS), J1.B4 (VBUS), J1.B9 (VBUS)
- net USB_D-: now reaches U2.53 (D-)
- net USB_D-: now also J1.A7 (D-), J1.B7 (D-)
- net USB_D+: now reaches U2.54 (D+)
- net USB_D+: now also J1.A6 (D+), J1.B6 (D+)
- net at R2.2: now also J1.A5 (CC1), J1.B5 (CC2)
- net at R6.2: now also U3.8
- new net: D1.1 (RK), R3.1
- new net: D1.2 (GK), R4.1
- new net: R4.2, U3.6
- new net: R11.2, U3.2
- new net: R9.2, U3.4
- new net: D2.1 (RK), R5.1
- new net: D2.2 (GK), R6.1
- new net: D3.1 (RK), R8.1
- new net: D3.2 (GK), R9.1
- new net: D4.1 (RK), R10.1
- new net: D4.2 (GK), R11.1
- no-connect marks 26 -> 14
Other:
- note added: "Barometric \nSensor"
- note added: "IMU"
- note added: "Microcontroller\n"
- note added: "USB"
- note removed: "Barometric Sensor"
- moved on the sheet: C1, C3, J2, J4, R1, R7, SW1, SW2, SW3, U1, U4, U5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

Commit message: PCB REV A
Parts:
- added BT1: Battery_Cell, Battery:BatteryHolder_Keystone_1060_1x2032, symbol Device:Battery_Cell
- added BZ1: Buzzer, Buzzer_Beeper:Buzzer_CUI_CPT-9019S-SMT, symbol Device:Buzzer
- added C7, C8, C9: 100nF, Capacitor_SMD:C_1206_3216Metric_Pad1.42x1.75mm_HandSolder, symbol Device:C
- added F1: Polyfuse, Fuse:Fuse_1812_4532Metric_Pad1.30x3.40mm_HandSolder, symbol Device:Polyfuse
- added J5: Conn_01x08, Connector_PinSocket_2.54mm:PinSocket_1x08_P2.54mm_Vertical, symbol Connector_Generic:Conn_01x08
- added R13: 11k, Resistor_SMD:R_1206_3216Metric_Pad1.42x1.75mm_HandSolder, symbol Device:R
- added R14: 10M, Resistor_SMD:R_1206_3216Metric_Pad1.42x1.75mm_HandSolder, symbol Device:R
- added R15: 3.3M, Resistor_SMD:R_1206_3216Metric_Pad1.42x1.75mm_HandSolder, symbol Device:R
- added SW4: SW_SPST, Button_Switch_SMD:SW_DIP_SPSTx01_Slide_6.7x4.1mm_W6.73mm_P2.54mm_LowProfile_JPin, symbol Switch:SW_SPST
- added TP1: TestPoint, Connector_Pin:Pin_D1.0mm_L10.0mm, symbol Connector:TestPoint
- added TP2, TP3, TP4: TestPoint, TestPoint:TestPoint_Loop_D2.50mm_Drill1.0mm, symbol Connector:TestPoint
- C3: footprint Capacitor_SMD:CP_Elec_10x10 -> Capacitor_SMD:CP_Elec_4x5.4
Connections:
- net +3V3: now also U7.2 (VCC_IO), C7.1, J5.1 (Pin_1), R13.2, TP3.1
- net +BATT: now also SW4.1 (A), TP4.1; no longer U5.1 (VI)
- net GND: now also BT1.2 (-), BZ1.2 (+), C7.2, C8.1, C9.1, J5.2 (Pin_2), R15.1, TP2.1
- net GPS_EXTINT: now reaches U2.21 (14_A0_TX3_SPDIF_OUT)
- net GPS_EXTINT: now also U7.19 (EXTINT)
- net BATT_SENSE: now reaches U2.22 (15_A1_RX3_SPDIF_IN)
- net BATT_SENSE: now also C9.2, R14.2, R15.2
- net SDA: now reaches U2.25 (18_A4_SDA0)
- net SDA: now also J5.4 (Pin_4)
- net SCL: now reaches U2.26 (19_A5_SCL0)
- net SCL: now also J5.3 (Pin_3)
- net BUZZER: now reaches U2.4 (2_OUT2)
- net BUZZER: now also BZ1.1 (-)
- net INT: now reaches U2.9 (7_RX2_OUT1A)
- net INT: now also J5.8 (Pin_8)
- net at SW3.2, U7.18 (~RESET): now also R13.1
- net at U7.3 (V_BCKP): now also BT1.1 (+), C8.2
- net at U7.8 (~SAFEBOOT): now also TP1.1
- new net: F1.1, R14.1, U5.1 (VI)
- new net: F1.2, SW4.2 (B)
- no-connect marks 14 -> 10
Other:
- moved on the sheet: C3, C5, J2, J4, SW3, U5, U7

Commit message: REV B
Parts:
- removed C3: 3.3uF, Capacitor_SMD:CP_Elec_4x5.4, symbol Device:CP1
- removed C6, C9: 100nF, Capacitor_SMD:C_1206_3216Metric_Pad1.42x1.75mm_HandSolder, symbol Device:C
- removed D1, D2, D3, D4: LED_RGBA, LED_SMD:LED_Avago_PLCC4_3.2x2.8mm_CW, symbol Device:LED_RGBA
- removed F1: Polyfuse, Fuse:Fuse_1812_4532Metric_Pad1.30x3.40mm_HandSolder, symbol Device:Polyfuse
- removed J4: Screw_Terminal_01x02, Connector_PinSocket_2.54mm:PinSocket_2x01_P2.54mm_Vertical, symbol Connector:Screw_Terminal_01x02
- removed J5: Conn_01x08, Connector_PinSocket_2.54mm:PinSocket_1x08_P2.54mm_Vertical, symbol Connector_Generic:Conn_01x08
- removed R10, R3, R5, R8: 51, Resistor_SMD:R_1206_3216Metric_Pad1.42x1.75mm_HandSolder, symbol Device:R
- removed R11, R4, R6, R9: 10, Resistor_SMD:R_1206_3216Metric_Pad1.42x1.75mm_HandSolder, symbol Device:R
- removed R14: 10M, Resistor_SMD:R_1206_3216Metric_Pad1.42x1.75mm_HandSolder, symbol Device:R
- removed R15: 3.3M, Resistor_SMD:R_1206_3216Metric_Pad1.42x1.75mm_HandSolder, symbol Device:R
- removed R2: R, Resistor_SMD:R_1206_3216Metric_Pad1.42x1.75mm_HandSolder, symbol Device:R
- removed SW4: SW_SPST, Button_Switch_SMD:SW_DIP_SPSTx01_Slide_6.7x4.1mm_W6.73mm_P2.54mm_LowProfile_JPin, symbol Switch:SW_SPST
- removed U1: ADIS16470AMLZ, footprints:ADIS16470AMLZ, symbol ADIS16470AMLZ:ADIS16470AMLZ
- removed U2: Teensy4.0, footprints:Teensy40, symbol teensy:Teensy4.0
- removed U3: 74LS14, Package_DIP:DIP-14_W7.62mm_SMDSocket_SmallPads, symbol 74xx:74LS14
- removed U4: RFM96W-433S2, RF_Module:HOPERF_RFM9XW_SMD, symbol RF_Module:RFM96W-433S2
- removed U5: LT1129-3.3_SOT223, Package_TO_SOT_SMD:SOT-223-3_TabPin2, symbol Regulator_Linear:LT1129-3.3_SOT223
- added C7: 3.3uF, Capacitor_SMD:CP_Elec_4x3.9, symbol Device:CP1
- added J1, J4: Conn_02x14_Counter_Clockwise, Connector_PinSocket_2.54mm:PinSocket_2x14_P2.54mm_Vertical, symbol Connector_Generic:Conn_02x14_Counter_Clockwise
- added J2: Conn_01x02, TerminalBlock:TerminalBlock_bornier-2_P5.08mm, symbol Connector_Generic:Conn_01x02
- added J3: Conn_02x08_Odd_Even, Connector_PinHeader_2.00mm:PinHeader_2x08_P2.00mm_Vertical_SMD, symbol Connector_Generic:Conn_02x08_Odd_Even
- added U1: RFM95W-915S2, RF_Module:HOPERF_RFM9XW_SMD, symbol RF_Module:RFM95W-915S2
- added U4: LT1129-3.3_SOT223, Package_TO_SOT_SMD:SOT-223-3_TabPin2, symbol Regulator_Linear:LT1129-3.3_SOT223
- renumbered C5 to C3, C7 to C5, C8 to C6, J1 to J5, J2 to J6, J3 to J7, R7 to R2, R13 to R3, R12 to R4, TP2 to TP1, TP3 to TP2, TP4 to TP3, TP1 to TP4, U6 to U2, U7 to U3
Connections:
- net +3V3: now also C7.1, J3.10 (Pin_10), J3.11 (Pin_11), J3.12 (Pin_12), J4.18 (Pin_18), J4.3 (Pin_3), U1.13 (3.3V), U4.3 (VO)
- net +BATT: now also J2.2 (Pin_2), U4.1 (VI)
- net BATT_SENSE: now also J4.12 (Pin_12)
- net BUZZER: now also J1.25 (Pin_25)
- net CS1:1: now also J1.17 (Pin_17)
- net CS1:2: now also J1.18 (Pin_18), J3.3 (Pin_3)
- net CS2: now also J1.27 (Pin_27), U1.5 (NSS)
- net GND: now also C7.2, J1.28 (Pin_28), J2.1 (Pin_1), J3.7 (Pin_7), J3.8 (Pin_8), J3.9 (Pin_9), J4.17 (Pin_17), J4.2 (Pin_2), J4.24 (Pin_24), J4.25 (Pin_25), U1.1 (GND), U1.10 (GND), U1.8 (GND), U4.2 (GND)
- net GPS_EXTINT: now also J4.13 (Pin_13)
- net IMU_DR: now also J1.19 (Pin_19), J3.13 (Pin_13)
- net INT: now also J1.20 (Pin_20)
- net MISO1: now also J1.15 (Pin_15), J3.4 (Pin_4)
- net MISO2: now also J1.26 (Pin_26), U1.2 (MISO)
- net MOSI1: now also J1.16 (Pin_16), J3.6 (Pin_6)
- net MOSI2: now also J4.21 (Pin_21), U1.3 (MOSI)
- net RX1: now also J4.11 (Pin_11)
- net SCK1: now also J3.2 (Pin_2), J4.14 (Pin_14)
- net SCK2: now also J4.23 (Pin_23), U1.4 (SCK)
- net SCL: now also J4.8 (Pin_8)
- net SDA: now also J4.9 (Pin_9)
- net SD_3.3: now also J1.5 (Pin_5)
- net SD_CLK: now also J1.4 (Pin_4)
- net SD_CMD: now also J1.6 (Pin_6)
- net SD_DAT0: now also J1.2 (Pin_2)
- net SD_DAT1: now also J1.1 (Pin_1)
- net SD_DAT2: now also J1.8 (Pin_8)
- net SD_DAT3: now also J1.7 (Pin_7)
- net SD_GND: now also J1.3 (Pin_3)
- net TX1: now also J4.10 (Pin_10)
- net USB_D+: now also J4.26 (Pin_26)
- net USB_D-: now also J4.27 (Pin_27)
- net V_USB: now also J4.28 (Pin_28)
- net at SW2.2: now also U1.6 (RESET)
- net at J7.1 (In): now also U1.9 (ANT)
- net at SW1.2: now also J3.1 (Pin_1)
- net at J5.A5 (CC1): no longer J5.B5 (CC2)
- new net on-off: J4.15 (Pin_15)
- new net pgm: J4.16 (Pin_16)
- new net vin: J4.1 (Pin_1)
- no-connect marks 10 -> 13
Other:
- note removed: "LED Indicators"
- moved on the sheet: BT1, BZ1, C1, C3, C5, C6, J6, R1, R3, SW1, SW3, TP1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
